File: Siddha-PCB/RocketryIN-FC.kicad_sch (KiCad schematic)
At the start: 2 parts, among them J1 Screw_Terminal_01x02, J2 Screw_Terminal_01x02

Commit message: switch to linear actuator and 7.4v battery
Connections:
- net +12V renamed +7.5V
Other:
- sheet Microcontoller ports: added LACTUATOR; removed SRVO1, SRVO2
- sheet Peripherals ports: added LACTUATOR; removed SRVO1, SRVO2
Changed lines of the file:
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@@
     (stroke (width 0) (type default))
   )
-  (wire (pts (xy 120.904 80.518) (xy 127 80.518))
+  (wire (pts (xy 120.65 80.518) (xy 127 80.518))
     (stroke (width 0) (type default))
   )
@@
     (stroke (width 0) (type default))
   )
-  (wire (pts (xy 120.904 85.598) (xy 127 85.598))
-    (stroke (width 0) (type default))
-  )
   (wire (pts (xy 120.65 104.902) (xy 127 104.902))
     (stroke (width 0) (type default))
   )
-  (wire (pts (xy 120.904 88.138) (xy 127 88.138))
-    (stroke (width 0) (type default))
-  )
   (wire (pts (xy 155.956 120.65) (xy 161.544 120.65))
     (stroke (width 0) (type default))
@@
     (stroke (width 0) (type default))
   )
-  (wire (pts (xy 120.904 75.438) (xy 127 75.438))
+  (wire (pts (xy 120.65 75.438) (xy 127 75.438))
     (stroke (width 0) (type default))
   )
@@
     (stroke (width 0) (type default))
   )
+  (wire (pts (xy 120.65 85.344) (xy 127 85.344))
+    (stroke (width 0) (type default))
+  )
   (wire (pts (xy 50.038 72.136) (xy 53.086 72.136))
     (stroke (width 0) (type default))
@@
     (stroke (width 0) (type default))
   )
-  (wire (pts (xy 120.904 77.978) (xy 127 77.978))
+  (wire (pts (xy 120.65 77.978) (xy 127 77.978))
     (stroke (width 0) (type default))
   )
@@
     (stroke (width 0) (type default))
   )
-  (wire (pts (xy 120.904 83.058) (xy 127 83.058))
+  (wire (pts (xy 120.65 83.058) (xy 127 83.058))
     (stroke (width 0) (type default))
   )
@@
   (hierarchical_label "BATT" (shape input) (at 53.594 48.768 0) (fields_autoplaced)
     (effects (font (size 1.27 1.27)) (justify left))
+  )
+  (symbol (lib_id "power:+7.5V") (at 53.086 68.834 0) (unit 1)
+    (in_bom yes) (on_board yes) (dnp no) (fields_autoplaced)
+    (property "Reference" "#PWR020" (at 53.086 72.644 0)
+      (effects (font (size 1.27 1.27)) hide)
+    )
+    (property "Value" "+7.5V" (at 53.086 63.5 0)
+      (effects (font (size 1.27 1.27)))
+    )
+    (property "Footprint" "" (at 53.086 68.834 0)
+      (effects (font (size 1.27 1.27)) hide)
+    )
+    (property "Datasheet" "" (at 53.086 68.834 0)
+      (effects (font (size 1.27 1.27)) hide)
+    )
+    (pin "1")
+    (instances
+      (project "RocketryIN-FC"
+        (path "/eca5bcb3-e8cc-4774-b734-f4245bf2d59b"
+          (reference "#PWR020") (unit 1)
+        )
+      )
+    )
   )
   (symbol (lib_id "Connector:Screw_Terminal_01x02") (at 45.466 51.308 180) (unit 1)
@@
     )
   )
-  (symbol (lib_id "power:+12V") (at 53.086 68.834 0) (unit 1)
-    (in_bom yes) (on_board yes) (dnp no)
-    (property "Reference" "#PWR022" (at 53.086 72.644 0)
-      (effects (font (size 1.27 1.27)) hide)
-    )
-    (property "Value" "+12V" (at 52.832 65.278 0)
-      (effects (font (size 1.27 1.27)))
-    )
-    (property "Footprint" "" (at 53.086 68.834 0)
-      (effects (font (size 1.27 1.27)) hide)
-    )
-    (property "Datasheet" "" (at 53.086 68.834 0)
-      (effects (font (size 1.27 1.27)) hide)
-    )
-    (pin "1")
-    (instances
-      (project "RocketryIN-FC"
-        (path "/eca5bcb3-e8cc-4774-b734-f4245bf2d59b"
-          (reference "#PWR022") (unit 1)
-        )
-      )
-    )
-  )
   (symbol (lib_id "power:GND") (at 53.594 52.832 0) (unit 1)
     (in_bom yes) (on_board yes) (dnp no) (fields_autoplaced)
@@
     )
   )
-  (sheet (at 104.394 73.66) (size 16.51 16.256)
-    (stroke (width 0.1524) (type solid))
-    (fill (color 0 0 0 0.0000))
-    (property "Sheetname" "Peripherals" (at 104.394 72.9484 0)
-      (effects (font (size 1.27 1.27)) (justify left bottom))
-    )
-    (property "Sheetfile" "peripherals.kicad_sch" (at 96.012 90.424 0)
-      (effects (font (size 1.27 1.27)) (justify left top))
-    )
-    (pin "BUZZ" input (at 120.904 83.058 0)
-      (effects (font (size 1.27 1.27)) (justify right))
-    )
-    (pin "SRVO1" input (at 120.904 85.598 0)
-      (effects (font (size 1.27 1.27)) (justify right))
-    )
-    (pin "SRVO2" input (at 120.904 88.138 0)
-      (effects (font (size 1.27 1.27)) (justify right))
-    )
-    (pin "BLUE" input (at 120.904 80.518 0)
-      (effects (font (size 1.27 1.27)) (justify right))
-    )
-    (pin "RED" input (at 120.904 75.438 0)
-      (effects (font (size 1.27 1.27)) (justify right))
-    )
-    (pin "GREEN" input (at 120.904 77.978 0)
+  (sheet (at 104.14 73.66) (size 16.51 16.256)
+    (stroke (width 0.1524) (type solid))
+    (fill (color 0 0 0 0.0000))
+    (property "Sheetname" "Peripherals" (at 104.14 72.9484 0)
+      (effects (font (size 1.27 1.27)) (justify left bottom))
+    )
+    (property "Sheetfile" "peripherals.kicad_sch" (at 95.758 90.424 0)
+      (effects (font (size 1.27 1.27)) (justify left top))
+    )
+    (pin "BUZZ" input (at 120.65 83.058 0)
+      (effects (font (size 1.27 1.27)) (justify right))
+    )
+    (pin "BLUE" input (at 120.65 80.518 0)
+      (effects (font (size 1.27 1.27)) (justify right))
+    )
+    (pin "RED" input (at 120.65 75.438 0)
+      (effects (font (size 1.27 1.27)) (justify right))
+    )
+    (pin "GREEN" input (at 120.65 77.978 0)
+      (effects (font (size 1.27 1.27)) (justify right))
+    )
+    (pin "LACTUATOR" input (at 120.65 85.344 0)
       (effects (font (size 1.27 1.27)) (justify right))
     )
@@
       (effects (font (size 1.27 1.27)) (justify left))
     )
-    (pin "SRVO2" input (at 127 88.138 180)
-      (effects (font (size 1.27 1.27)) (justify left))
-    )
-    (pin "SRVO1" input (at 127 85.598 180)
-      (effects (font (size 1.27 1.27)) (justify left))
-    )
     (pin "BLUE" input (at 127 80.518 180)
       (effects (font (size 1.27 1.27)) (justify left))
@@
       (effects (font (size 1.27 1.27)) (justify left))
     )
+    (pin "LACTUATOR" input (at 127 85.344 180)
+      (effects (font (size 1.27 1.27)) (justify left))
+    )
